File: Desk_controller.kicad_pcb (KiCad board)
At the start: 2 copper layers, 100 x 51.2 mm, 4 parts

Commit message: starting project migration
Parts:
- added C1: 100n, Capacitor_SMD:C_0603_1608Metric_Pad1.08x0.95mm_HandSolder, F.Cu at (109.3, 85.1)
- added C10: 22p, Capacitor_SMD:C_0603_1608Metric_Pad1.08x0.95mm_HandSolder, F.Cu at (135.0, 57.5)
- added C11: 1u, Capacitor_SMD:C_0603_1608Metric_Pad1.08x0.95mm_HandSolder, F.Cu at (138.0, 59.5)
- added C12: 33p, Capacitor_SMD:C_0603_1608Metric_Pad1.08x0.95mm_HandSolder, F.Cu at (162.9, 83.9)
- added C13: 100n, Capacitor_SMD:C_0603_1608Metric_Pad1.08x0.95mm_HandSolder, F.Cu at (138.0, 61.3)
- added C14: 22p, Capacitor_SMD:C_0603_1608Metric_Pad1.08x0.95mm_HandSolder, F.Cu at (132.0, 53.9)
- added C15: 22u, Capacitor_SMD:C_1210_3225Metric_Pad1.33x2.70mm_HandSolder, F.Cu at (175.9, 78.8)
- added C16: 1u, Capacitor_SMD:C_0603_1608Metric_Pad1.08x0.95mm_HandSolder, F.Cu at (125.6, 71.9)
- added C17: 22u, Capacitor_SMD:C_1210_3225Metric_Pad1.33x2.70mm_HandSolder, F.Cu at (170.6, 78.8)
- added C18: 22u, Capacitor_SMD:C_1210_3225Metric_Pad1.33x2.70mm_HandSolder, F.Cu at (170.6, 75.5)
- added C19: 100n, Capacitor_SMD:C_0603_1608Metric_Pad1.08x0.95mm_HandSolder, F.Cu at (127.4, 71.9)
- added C2: 4.7u, Capacitor_SMD:C_1206_3216Metric_Pad1.33x1.80mm_HandSolder, F.Cu at (171.6, 71.1)
- added C20: 100n, Capacitor_SMD:C_0603_1608Metric_Pad1.08x0.95mm_HandSolder, F.Cu at (125.6, 68.4)
- added C21: 1n, Capacitor_SMD:C_0603_1608Metric_Pad1.08x0.95mm_HandSolder, F.Cu at (123.6, 54.1)
- added C22: 1n, Capacitor_SMD:C_0603_1608Metric_Pad1.08x0.95mm_HandSolder, F.Cu at (142.1, 47.0)
- added C23: 1n, Capacitor_SMD:C_0603_1608Metric_Pad1.08x0.95mm_HandSolder, F.Cu at (145.4, 50.3)
- added C24: 220u, Capacitor_SMD:CP_Elec_10x10, F.Cu at (171.1, 60.8)
- added C25: 100n, Capacitor_SMD:C_0603_1608Metric_Pad1.08x0.95mm_HandSolder, F.Cu at (149.2, 60.5)
- added C26: 10n, Capacitor_SMD:C_0603_1608Metric_Pad1.08x0.95mm_HandSolder, F.Cu at (142.1, 43.5)
- added C27: 10n, Capacitor_SMD:C_0603_1608Metric_Pad1.08x0.95mm_HandSolder, F.Cu at (149.0, 50.3)
- added C3: 10n, Capacitor_SMD:C_0603_1608Metric_Pad1.08x0.95mm_HandSolder, F.Cu at (120.8, 80.8)
- added C4: 4.7u, Capacitor_SMD:C_1206_3216Metric_Pad1.33x1.80mm_HandSolder, F.Cu at (169.0, 71.2)
- added C5: 10n, Capacitor_SMD:C_0603_1608Metric_Pad1.08x0.95mm_HandSolder, F.Cu at (129.7, 80.8)
- added C6: 100n, Capacitor_SMD:C_0603_1608Metric_Pad1.08x0.95mm_HandSolder, F.Cu at (165.7, 70.9)
- added C7: 1n, Capacitor_SMD:C_0603_1608Metric_Pad1.08x0.95mm_HandSolder, F.Cu at (124.3, 80.8)
- added C8: 1n, Capacitor_SMD:C_0603_1608Metric_Pad1.08x0.95mm_HandSolder, F.Cu at (126.1, 80.8)
- added C9: 100n, Capacitor_SMD:C_0603_1608Metric_Pad1.08x0.95mm_HandSolder, F.Cu at (165.2, 81.3)
- added D1: BAV99, Package_TO_SOT_SMD:SOT-23, F.Cu at (126.4, 54.1)
- added J1: B4B XH A, Connector_JST:JST_XH_B4B-XH-A_1x04_P2.50mm_Vertical, F.Cu at (121.6, 86.4)
- added J2: 01x04 socket, Connector_PinSocket_2.54mm:PinSocket_1x04_P2.54mm_Vertical, B.Cu at (182.4, 69.5)
- added J3: 01x14 socket, Connector_PinSocket_2.54mm:PinSocket_1x14_P2.54mm_Vertical, B.Cu at (109.2, 82.2)
- added J4: HX JN1.27-2x5 WZ H4.9, Personal:JN1.27-2x5 WZ H4.9, B.Cu at (148.2, 81.9)
- added J5: USB_C_Receptacle_USB2.0_16P, Personal:USB_C_socket_16P_vertical, F.Cu at (138.0, 84.1)
- added J6: Dell DC jack, Personal:Dell DC jack, F.Cu at (193.7, 90.7)
- added J7: B6B XH A, Connector_JST:JST_XH_B6B-XH-A_1x06_P2.50mm_Vertical, F.Cu at (159.9, 45.1)
- added J8: DC barrel assy, Personal:Dell_barrel_assy, F.Cu at (171.1, 52.1)
- added JP1: 0R, Personal:Jumper_0603, F.Cu at (113.4, 51.4)
- added JP10: 0R, Personal:Jumper_0603, F.Cu at (113.4, 74.5)
- added JP11: 0R, Personal:Jumper_0603, F.Cu at (113.4, 77.0)
- added JP12: 0R, Personal:Jumper_0603, F.Cu at (180.0, 74.2)
- added JP13: 0R, Personal:Jumper_0603, F.Cu at (123.8, 71.9)
- added JP14: 0R, Resistor_SMD:R_1206_3216Metric_Pad1.30x1.75mm_HandSolder, F.Cu at (148.2, 70.7)
- added JP15: 0R, Personal:Jumper_0603, F.Cu at (144.4, 65.6)
- added JP16: 0R, Personal:Jumper_0603, F.Cu at (144.4, 67.6)
- added JP17: 0R, Personal:Jumper_0603, F.Cu at (144.4, 69.6)
- added JP18: 0R, Resistor_THT:R_Axial_DIN0204_L3.6mm_D1.6mm_P7.62mm_Horizontal, F.Cu at (160.1, 58.5)
- added JP19: 0R, Resistor_SMD:R_1206_3216Metric_Pad1.30x1.75mm_HandSolder, F.Cu at (143.4, 54.7)
- added JP2: 0R, Personal:Jumper_0603, F.Cu at (113.4, 53.1)
- added JP20: 0R, Resistor_SMD:R_0603_1608Metric_Pad0.98x0.95mm_HandSolder, F.Cu at (133.2, 80.8)
- added JP21: 0R, Personal:Jumper_0603, F.Cu at (138.0, 78.0)
- added JP22: 0R, Resistor_THT:R_Axial_DIN0204_L3.6mm_D1.6mm_P7.62mm_Horizontal, F.Cu at (162.3, 56.7)
- added JP23: 0R, Personal:Wire_9.603mm, B.Cu at (151.6, 56.6)
- added JP24: 0R, Personal:Wire_6.310mm, B.Cu at (152.8, 63.2)
- added JP25: 0R, Personal:Wire_9.532mm, B.Cu at (134.1, 67.4)
- added JP26: 0R, Personal:Wire_6.853x8.890mm, F.Cu at (136.1, 68.2)
- added JP3: 0R, Personal:Jumper_0603, F.Cu at (113.4, 54.9)
- added JP4: 0R, Resistor_SMD:R_1206_3216Metric_Pad1.30x1.75mm_HandSolder, F.Cu at (114.2, 57.2)
- added JP5: 0R, Resistor_SMD:R_1206_3216Metric_Pad1.30x1.75mm_HandSolder, F.Cu at (114.2, 59.7)
- added JP6: 0R, Resistor_SMD:R_0603_1608Metric_Pad0.98x0.95mm_HandSolder, F.Cu at (113.4, 62.0)
- added JP7: 0R, Resistor_SMD:R_1206_3216Metric_Pad1.30x1.75mm_HandSolder, F.Cu at (114.2, 66.3)
- added JP8: 0R, Personal:Jumper_0603, F.Cu at (113.4, 69.4)
- added JP9: 0R, Resistor_THT:R_Axial_DIN0204_L3.6mm_D1.6mm_P5.08mm_Horizontal, F.Cu at (120.3, 62.3)
- added L1: 10u, Personal:L_Bourns_SRP6540, F.Cu at (170.1, 84.1)
- added R10: 2k2, Resistor_SMD:R_0603_1608Metric_Pad0.98x0.95mm_HandSolder, F.Cu at (123.6, 50.3)
- added R11: 820, Resistor_SMD:R_0603_1608Metric_Pad0.98x0.95mm_HandSolder, F.Cu at (125.3, 50.3)
- added R12: 2k2, Resistor_SMD:R_0603_1608Metric_Pad0.98x0.95mm_HandSolder, F.Cu at (147.2, 50.3)
- added R13: 2k2, Resistor_SMD:R_0603_1608Metric_Pad0.98x0.95mm_HandSolder, F.Cu at (142.1, 45.3)
- added R14: 5k1, Resistor_SMD:R_0603_1608Metric_Pad0.98x0.95mm_HandSolder, F.Cu at (134.2, 86.2)
- added R15: 5k1, Resistor_SMD:R_0603_1608Metric_Pad0.98x0.95mm_HandSolder, F.Cu at (141.9, 82.1)
- added R5: 2k2, Resistor_SMD:R_0603_1608Metric_Pad0.98x0.95mm_HandSolder, F.Cu at (122.6, 80.8)
- added R6: 23.2k, Resistor_SMD:R_0603_1608Metric_Pad0.98x0.95mm_HandSolder, F.Cu at (161.2, 83.9)
- added R7: 10k, Resistor_SMD:R_0603_1608Metric_Pad0.98x0.95mm_HandSolder, F.Cu at (161.2, 77.8)
- added R8: 10k, Resistor_SMD:R_0603_1608Metric_Pad0.98x0.95mm_HandSolder, F.Cu at (129.4, 54.4)
- added R9: 10k, Resistor_SMD:R_0603_1608Metric_Pad0.98x0.95mm_HandSolder, F.Cu at (139.3, 55.7)
- added TFT1: TFT_2.4in_320x240, Personal:Display_240x320_ILI9341_2.4in_no_pads, B.Cu at (145.8, 65.7)
- added TP1: TestPoint, TestPoint:TestPoint_THTPad_D1.0mm_Drill0.5mm, F.Cu at (163.4, 80.8)
- added TP10: TestPoint, TestPoint:TestPoint_THTPad_D1.0mm_Drill0.5mm, F.Cu at (176.7, 71.9)
- added TP11: TestPoint, TestPoint:TestPoint_THTPad_D1.0mm_Drill0.5mm, F.Cu at (137.3, 70.9)
- added TP12: TestPoint, TestPoint:TestPoint_THTPad_D1.0mm_Drill0.5mm, F.Cu at (144.7, 57.2)
- added TP13: TestPoint, TestPoint:TestPoint_THTPad_D1.0mm_Drill0.5mm, F.Cu at (142.1, 57.2)
- added TP14: TestPoint, TestPoint:TestPoint_THTPad_D1.0mm_Drill0.5mm, F.Cu at (121.5, 51.4)
- added TP15: TestPoint, TestPoint:TestPoint_THTPad_D1.0mm_Drill0.5mm, F.Cu at (147.2, 54.7)
- added TP16: TestPoint, TestPoint:TestPoint_THTPad_D1.0mm_Drill0.5mm, F.Cu at (142.1, 88.2)
- added TP17: TestPoint, TestPoint:TestPoint_THTPad_D1.0mm_Drill0.5mm, F.Cu at (182.8, 77.5)
- added TP18: TestPoint, TestPoint:TestPoint_THTPad_D1.0mm_Drill0.5mm, F.Cu at (182.8, 79.8)
- added TP19: TestPoint, TestPoint:TestPoint_THTPad_D1.0mm_Drill0.5mm, F.Cu at (121.5, 53.9)
- added TP2: TestPoint, TestPoint:TestPoint_THTPad_D1.0mm_Drill0.5mm, F.Cu at (162.7, 70.9)
- added TP20: TestPoint, TestPoint:TestPoint_THTPad_D1.0mm_Drill0.5mm, F.Cu at (164.7, 87.9)
- added TP21: TestPoint, TestPoint:TestPoint_THTPad_D1.0mm_Drill0.5mm, F.Cu at (147.2, 56.9)
- added TP3: TestPoint, TestPoint:TestPoint_THTPad_D1.0mm_Drill0.5mm, F.Cu at (126.4, 77.8)
- added TP4: TestPoint, TestPoint:TestPoint_THTPad_D1.0mm_Drill0.5mm, F.Cu at (124.1, 77.8)
- added TP5: TestPoint, TestPoint:TestPoint_THTPad_D1.0mm_Drill0.5mm, F.Cu at (161.2, 80.8)
- added TP6: TestPoint, TestPoint:TestPoint_THTPad_D1.0mm_Drill0.5mm, F.Cu at (165.0, 84.1)
- added TP7: TestPoint, TestPoint:TestPoint_THTPad_D1.0mm_Drill0.5mm, F.Cu at (120.8, 76.5)
- added TP8: TestPoint, TestPoint:TestPoint_THTPad_D1.0mm_Drill0.5mm, F.Cu at (139.6, 72.7)
- added TP9: TestPoint, TestPoint:TestPoint_THTPad_D1.0mm_Drill0.5mm, F.Cu at (141.4, 61.3)
- added U1: LMR38020, Package_SO:Texas_HSOP-8-1EP_3.9x4.9mm_P1.27mm_ThermalVias, F.Cu at (165.0, 75.7)
- added U2: STM32G431K8T, Package_QFP:LQFP-32_7x7mm_P0.8mm, F.Cu at (132.2, 65.8)
- added U3: VNH7070, Package_SO:JEITA_SOIC-16_3.9x9.9mm_P1.27mm, F.Cu at (155.1, 60.5)
- added U4: USBLC6-2SC6, Package_TO_SOT_SMD:SOT-23-6, F.Cu at (134.5, 76.8)
- added Y1: 20 MHz, Crystal:Crystal_SMD_3225-4Pin_3.2x2.5mm_HandSoldering, F.Cu at (135.0, 53.9)
- R1: value 10 -> 10k
- R2: value 100 -> 10k
- R3: value 200 -> 64.9k
- R4: value 300 -> 2k2
- moved R1 1.50 mm to (119.0, 80.8)
- moved R2 1.50 mm to (131.4, 80.8)
- moved R3 1.50 mm to (161.2, 73.7)
- moved R4 1.50 mm to (127.9, 80.8)
Connections:
- R1 pad 1: /System overview/Block diagram/Childsheet_1_example/Signal2 -> /System overview/Block diagram/S3V3
- R1 pad 2: GND -> /System overview/Block diagram/Limit switch interface/BOT_EOT
- R2 pad 1: /System overview/Block diagram/Childsheet_1_example/Signal1 -> /System overview/Block diagram/S3V3
- R2 pad 2: GND -> /System overview/Block diagram/Limit switch interface/TOP_EOT
- R3 pad 1: /System overview/Block diagram/Childsheet_1_example/Signal1 -> /System overview/Block diagram/DCDC converter 3V3/RT
- R3 pad 2: GND -> /System overview/Block diagram/GND
- R4 pad 1: /System overview/Block diagram/Childsheet_1_example/Signal2 -> /System overview/Block diagram/Limit switch interface/TOP_EOT
- R4 pad 2: GND -> /System overview/Block diagram/Limit switch interface/TOP_filt
Routing:
- net /System overview/Block diagram/S3V3: track 0.00 -> 369.3 mm
- net /System overview/Block diagram/GND: track 0.00 -> 58.2 mm, vias 0 -> 62
- net /System overview/Block diagram/Childsheet_1_example/Signal1: track 47.3 -> 0.00 mm
- net GND: track 46.2 -> 0.00 mm, vias 1 -> 0
- net /System overview/Block diagram/Display/DISP_MOSI: track 0.00 -> 31.3 mm
- net /System overview/Block diagram/Display/DISP_MISO: track 0.00 -> 31.2 mm
- net /System overview/Block diagram/Microcontroller/SWDIO: track 0.00 -> 26.6 mm
- net /System overview/Block diagram/Microcontroller/ENCb_filt: track 0.00 -> 25.8 mm
- net /System overview/Block diagram/Servomotor interface/SEL0': track 0.00 -> 25.8 mm
- net /System overview/Block diagram/DCDC converter 3V3/3V3_REG: track 0.00 -> 23.9 mm
- net /System overview/Block diagram/Microcontroller/ENCa_filt: track 0.00 -> 23.8 mm
- net Net-(JP19-Pad1): track 0.00 -> 22.5 mm
- net /System overview/Block diagram/Microcontroller/SWDCLK: track 0.00 -> 22.4 mm
- net /System overview/Block diagram/Display/TCH_IRQ: track 0.00 -> 21.0 mm
- net /System overview/Block diagram/S19V5: track 0.00 -> 20.0 mm, vias 0 -> 4
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- added copper zone on F.Cu, net (none)
- added copper zone on F.Cu, net /System overview/Block diagram/DCDC converter 3V3/3V3_REG
- added copper zone on F.Cu, net /System overview/Block diagram/DCDC converter 3V3/GND_2
- added copper zone on B.Cu, net /System overview/Block diagram/DCDC converter 3V3/S19V5_2
- added copper zone on F.Cu, net /System overview/Block diagram/DCDC converter 3V3/SW
- added copper zone on B.Cu, net /System overview/Block diagram/GND
- added copper zone on F.Cu, net /System overview/Block diagram/GND
- added copper zone on B.Cu, net /System overview/Block diagram/S19V5
- added copper zone on F.Cu, net /System overview/Block diagram/S19V5
- added copper zone on F.Cu, net /System overview/Block diagram/Servomotor interface/OUTa
- added copper zone on F.Cu, net /System overview/Block diagram/Servomotor interface/OUTb
- added copper zone on F.Cu, net /System overview/Block diagram/Servomotor interface/OUTb'
- removed copper zone on B.Cu, net GND
Other:
- outline, holes or cut-outs redrawn
- board text added: "23/09/2026"
- board text added: "3V3_REG"
- board text added: "BOT"
- board text added: "CS"
- board text added: "Cut here"
- board text added: "ENCa"
- board text added: "ENCb"
- board text added: "Felipe L Rodrigues"
- board text added: "Limit sw"
- board text added: "MOT_CS"
- board text added: "Motor"
- board text added: "PWR in"
- board text added: "S3V3"
- board text added: "TOP"
- board text added: "Table controller"
