File: Desk_controller.kicad_pcb (KiCad board)
At the start: 2 copper layers, 100 x 51.2 mm, 105 parts, among them J1 B4B XH A, J2 01x04 socket, J3 01x14 socket, J4 HX JN1.27-2x5 WZ H4.9, J5 USB_C_Receptacle_USB2.0_16P, J6 Dell DC jack, J7 B6B XH A, J8 DC barrel assy, U1 LMR380x0, U2 STM32G431K8T, U3 VNH7070, U4 USBLC6-2SC6, Y1 20 MHz

Commit message: add TP layer
Other:
- board text added: "BOOT0"
- board text added: "BOT_filt"
- board text added: "ENCa_filt"
- board text added: "ENCb_filt"
- board text added: "FB"
- board text added: "NRST"
- board text added: "PG"
- board text added: "RT"
- board text added: "SEL0"
- board text added: "SW"
- board text added: "TOP_filt"
- board text added: "VBUS"
