File: Block_diagram.kicad_sch (KiCad schematic)
At the start: 0 parts

Commit message: starting project migration
Other:
- sheet Childsheet_1_example renamed Microcontroller
- sheet Childsheet_2_example renamed Servomotor interface
- added sheet DCDC converter 3V3 (DCDC_converter_3V3.kicad_sch)
- added sheet Display (Display.kicad_sch)
- added sheet Limit switch interface (Limit_switch_interface.kicad_sch)
- sheet Microcontroller: file Childsheet_1_example.kicad_sch -> Microcontroller.kicad_sch
- sheet Microcontroller ports: added BOT_filt, DISP_CS, DISP_DC, DISP_MISO, DISP_MOSI, DISP_RST, DISP_SCK, ENCa_filt, ENCb_filt, GND, INa, INb, MOT_CS, PWM, S3V3, SEL0, TCH_CS, TCH_IRQ, TOP_filt; removed Signal1, Signal2
- sheet Servomotor interface: file Childsheet_2_example.kicad_sch -> Servomotor_interface.kicad_sch
- sheet Servomotor interface ports: added ENCa_filt, ENCb_filt, GND, INa, INb, MOT_CS, PWM, S19V5, S3V3, SEL0; removed Signal1, Signal2
