File: DCDC_converter_3V3.kicad_sch (KiCad schematic)
At the start: 24 parts, among them J6 Dell DC jack, J8 DC barrel assy, U1 LMR38020

Commit message: refining fab and assy docs
Parts:
- U1: value LMR38020 -> LMR380x0; footprint Package_SO:Texas_HSOP-8-1EP_3.9x4.9mm_P1.27mm_ThermalVias -> Personal:Texas_HSOP-8-1EP_3.9x4.9mm_P1.27mm_ThermalVias_w_step
Changed lines of the file:
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@@
 			)
 		)
-		(property "Value" "LMR38020"
+		(property "Value" "LMR380x0"
 			(at 120.65 66.04 0)
 			(show_name no)
@@
 			)
 		)
-		(property "Footprint" "Package_SO:Texas_HSOP-8-1EP_3.9x4.9mm_P1.27mm_ThermalVias"
+		(property "Footprint" "Personal:Texas_HSOP-8-1EP_3.9x4.9mm_P1.27mm_ThermalVias_w_step"
 			(at 133.35 85.09 0)
 			(hide yes)
