File: Desk_controller.kicad_sch (KiCad schematic)
At the start: 0 parts

Commit message: starting project migration
Other:
- note added: "Migration to FLRHW KiCad starter template"
- note removed: "Description example"
- note removed: "TBD"

Commit message: add TP layer
Other:
- note removed: "${SHEET_TITLE_12}"
- note removed: "11"
- note removed: "12"
- note removed: "13"
- note removed: "14"
- note removed: "15"
- note removed: "16"
- note removed: "17"
- note removed: "18"
- note removed: "19"
- note removed: "21"
- note removed: "22"
- note removed: "23"
- note removed: "24"
- note removed: "25"
- note removed: "26"
- note removed: "27"
- note removed: "28"
- note removed: "29"
- note removed: "30"
- title: PROJECT TITLE -> Desk controller

Commit message: ready for release
Other:
- note added: "16/10/2026"
- note removed: "18/10/2026"
Changed lines of the file:
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@@
 		)
 	)
-	(text "18/10/2026"
+	(text "16/10/2026"
 		(exclude_from_sim no)
 		(at 102.235 44.45 0)

Commit message: Document revision 1.1.1: container CI and Pages publishing
Other:
- note added: "1.1.1"
- note added: "21/10/2026"
- note added: "Template updates: 1) CI now uses a single container; 2) added GitHub Pages publishing"
Changed lines of the file:
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@@
 	(title_block
 		(title "Desk controller")
-		(date "2026-10-18")
-		(rev "1.1.0")
+		(date "2026-10-21")
+		(rev "1.1.1")
 	)
 	(text "Table of contents"
@@
 		)
 	)
+	(text "21/10/2026"
+		(exclude_from_sim no)
+		(at 102.235 49.53 0)
+		(effects
+			(font
+				(face "DejaVu Sans")
+				(size 2.032 2.032)
+				(thickness 0.3175)
+				(color 0 0 0 1)
+			)
+			(justify left top)
+		)
+	)
 	(text "1.1.0"
 		(exclude_from_sim no)
@@
 		)
 	)
+	(text "1.1.1"
+		(exclude_from_sim no)
+		(at 89.535 49.53 0)
+		(effects
+			(font
+				(face "DejaVu Sans")
+				(size 2.032 2.032)
+				(thickness 0.3175)
+				(color 0 0 0 1)
+			)
+			(justify left top)
+		)
+	)
 	(text "${SHEET_TITLE_6}"
 		(exclude_from_sim no)
@@
 		)
 	)
+	(text "Template updates: 1) CI now uses a single container; 2) added GitHub Pages publishing"
+		(exclude_from_sim no)
+		(at 123.825 49.53 0)
+		(effects
+			(font
+				(face "DejaVu Sans")
+				(size 2.032 2.032)
+				(thickness 0.3175)
+				(color 0 0 0 1)
+			)
+			(justify left top)
+		)
+	)
