File: Interface_Power_supply.kicad_sch (KiCad schematic)
At the start: 0 parts

Commit message: starting project migration
Other:
- note added: "Barrel connector (Dell type, with ID pin) Pin 1 Supply - 19.5 V, 3 A (inner shell) 2 ID (internal pin) 3 GND (outer shell) SH Shield"
- note removed: "List here the requirements for the interface to the external world, e.g., connector type, pin definition."
Changed lines of the file:
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@@
 	(paper "A4")
 	(title_block
-		(date "2026-10-06")
-		(rev "1.0.0")
+		(date "2026-10-18")
+		(rev "1.1.0")
 	)
-	(text "List here the requirements for the interface to the external world, e.g., connector type, pin definition."
+	(text "Barrel connector (Dell type, with ID pin)\n\nPin \n  1  Supply - 19.5 V, 3 A (inner shell)\n  2  ID (internal pin)\n  3  GND (outer shell)\n SH  Shield"
 		(exclude_from_sim no)
 		(at 26.035 31.75 0)
