File: Microcontroller.kicad_sch (KiCad schematic)
At the start: 70 parts, among them J4 HX JN1.27-2x5 WZ H4.9, J5 USB_C_Receptacle_USB2.0_16P, U2 STM32G431K8T, U4 USBLC6-2SC6, Y1 20 MHz

Commit message: erc clear
Parts:
- J5: symbol Connector:USB_C_Receptacle_USB2.0_16P -> personal:USB_C_Receptacle_USB2.0_16P
Changed lines of the file:
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@@
 	)
 	(symbol
-		(lib_id "Connector:USB_C_Receptacle_USB2.0_16P")
+		(lib_id "personal:USB_C_Receptacle_USB2.0_16P")
 		(at 209.55 76.2 0)
 		(unit 1)
