File: System_overview.kicad_sch (KiCad schematic)
At the start: 0 parts

Commit message: starting project migration
Other:
- sheet Interface_childsheet_0_example renamed Servomotor
- added sheet DC power supply (Interface_Power_supply.kicad_sch)
- added sheet Limit switches (Interface_Limit_switches.kicad_sch)
- sheet Servomotor: file Interface_childsheet_0_example.kicad_sch -> Interface_servomotor.kicad_sch
- note added: "AC / DC"
- note added: "Bottom"
- note added: "DCDC converter Control logic Servomotor interface (power driver + encoder conditioning) Limit switch interface Display"
- note added: "DESK MECHANISM"
- note added: "Motor, gearbox and encoder"
- note added: "Top"
- note removed: "Simple description of contents"
- title: (none) -> Desk controller

Commit message: add TP layer
Other:
- title: Desk controller -> (none)
Changed lines of the file:
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@@
 	(paper "A4")
 	(title_block
-		(title "Desk controller")
 		(date "2026-10-18")
 		(rev "1.1.0")
